Commit message: added left wheel

File: src/bumper_bot_description/urdf/bumperbot.urdf.xacro (robot description, xacro)
@@ -17,12 +17,16 @@
         <origin xyz="0 0 0.033" rpy="0 0 0"/>
     </joint>
-    <link>
-        <name>laser_link</name>
+    <link name="left_wheel_link">
         <visual>
             <geometry>
-                <mesh filename="package://bumper_bot_description/meshes/laser.STL"/>
+                <mesh filename="package://bumper_bot_description/meshes/caster_front_link.STL"/>
             </geometry>
-            <origin xyz="0 0 0.1" rpy="0 0 0"/>
+            <origin xyz="0 0 0" rpy="0 0 0"/>
         </visual>
     </link>
+    <joint name="left_wheel_joint" type="fixed">
+        <parent link="base_link"/>
+        <child link="left_wheel_link"/>
+        <origin xyz="0.33 0 0" rpy="0 0 0"/>
+    </joint>
 </robot>

Commit message: final urdf file bumperbot

File: src/bumper_bot_description/urdf/bumperbot.urdf.xacro (robot description, xacro)
@@ -20,4 +20,31 @@
         <visual>
             <geometry>
+                <mesh filename="package://bumper_bot_description/meshes/wheel_left_link.STL"/>
+            </geometry>
+            <origin xyz="0 0 0" rpy="-1.57 0 0"/>
+        </visual>
+    </link>
+    <joint name="left_wheel_joint" type="continuous">
+        <parent link="base_link"/>
+        <child link="left_wheel_link"/>
+        <axis xyz="0.0 1.0 0.0"/>
+        <origin xyz="0 0.07 0" rpy="0 0 0"/>
+    </joint>
+  <link name="right_wheel_link">
+        <visual>
+            <geometry>
+                <mesh filename="package://bumper_bot_description/meshes/wheel_right_link.STL"/>
+            </geometry>
+            <origin xyz="0 0 0" rpy="1.57 0 0"/>
+        </visual>
+    </link>
+    <joint name="right_wheel_joint" type="continuous">
+        <parent link="base_link"/>
+        <child link="right_wheel_link"/>
+        <origin xyz="0 -0.07 0" rpy="0 0 0"/>
+    </joint>
+    <link name="castor_front_link">
+        <visual>
+            <geometry>
                 <mesh filename="package://bumper_bot_description/meshes/caster_front_link.STL"/>
             </geometry>
@@ -25,8 +52,21 @@
         </visual>
     </link>
-    <joint name="left_wheel_joint" type="fixed">
+    <joint name="castor_front_joint" type="fixed">
         <parent link="base_link"/>
-        <child link="left_wheel_link"/>
-        <origin xyz="0.33 0 0" rpy="0 0 0"/>
+        <child link="castor_front_link"/>
+        <origin xyz="0.04755 0 -0.0275" rpy="0 0 0"/>
+    </joint>
+    <link name="castor_back_link">
+        <visual>
+            <geometry>
+                <mesh filename="package://bumper_bot_description/meshes/caster_rear_link.STL"/>
+            </geometry>
+            <origin xyz="0 0 0" rpy="0 0 0"/>
+        </visual>
+    </link>
+    <joint name="castor_back_joint" type="fixed">
+        <parent link="base_link"/>
+        <child link="castor_back_link"/>
+        <origin xyz="-0.04755 0 -0.0275" rpy="0 0 0"/>
     </joint>
 </robot>

Commit message: added launch files to the tutorial section

File: src/bumper_bot_description/urdf/bumperbot.urdf.xacro (robot description, xacro)
@@ -42,4 +42,5 @@
         <parent link="base_link"/>
         <child link="right_wheel_link"/>
+        <axis xyz="0.0 1.0 0.0"/>
         <origin xyz="0 -0.07 0" rpy="0 0 0"/>
     </joint>

Commit message: launch lecture completed

File: src/bumper_bot_description/urdf/bumperbot.urdf.xacro (robot description, xacro)
@@ -1,4 +1,5 @@
 <?xml version="1.0"?>
 <robot name="bumperbot" xmlns:xacro="http://www.ros.org/wiki/xacro">
+    <xacro:include filename="$(find bumper_bot_description)/urdf/bumperbot_gazebo.xacro"/>
     <link name="base_footprint">
     </link>
@@ -11,4 +12,17 @@
             <origin xyz="0 0 0" rpy="0 0 0"/>
         </visual>
+        <collision>
+            <geometry>
+                <mesh filename="package://bumper_bot_description/meshes/base_link.STL"/>
+            </geometry>
+            <origin xyz="0 0 0" rpy="0 0 0"/>
+        </collision>
+        <inertial>
+            <origin xyz="0 0 0.04" rpy="0.0 0.25 0.3"/>
+            <mass value="8.2573504e-01"/>
+            <inertia ixx="2.2124416e-02" ixy="-1.2294101e-04"
+                     ixz="3.4938785e-04" iyy="2.1193702e-02"
+                     iyz="-5.0120904e-05" izz="2.0064271e-02"/>
+        </inertial>
     </link>
     <joint name="base_joint" type="fixed">
@@ -24,4 +38,17 @@
             <origin xyz="0 0 0" rpy="-1.57 0 0"/>
         </visual>
+        <collision>
+            <origin xyz="0 0.015 0" rpy="1.57 0 0"/>
+            <geometry>
+                <cylinder radius="0.033" length="0.01"/>
+            </geometry>
+        </collision>
+        <inertial>
+            <origin xyz="0 -0.014 0" rpy="0 0 0"/>
+            <mass value="0.0530086090966721"/>
+            <inertia ixx="1.8792911368909E-05" ixy="3.31256392204584E-10"
+                    ixz="-1.14082001662767E-08" iyy="3.11510738759073E-05"
+                    iyz="-3.60499245082192E-10" izz="1.88266886146847E-05"/>
+        </inertial>
     </link>
     <joint name="left_wheel_joint" type="continuous">
@@ -38,4 +65,17 @@
             <origin xyz="0 0 0" rpy="1.57 0 0"/>
         </visual>
+        <collision>
+            <origin xyz="0 -0.015 0" rpy="1.57 0 0"/>
+            <geometry>
+                <cylinder radius="0.033" length="0.01"/>
+            </geometry>
+        </collision>
+        <inertial>
+            <origin xyz="0 -0.014 0" rpy="0 0 0"/>
+            <mass value="0.0530086090966721"/>
+            <inertia ixx="1.88176298336665E-05" ixy="-4.8444933029987E-10"
+                    ixz="1.88163708851143E-08" iyy="3.11510738647764E-05"
+                    iyz="-6.93560663069607E-11" izz="1.8801969558182E-05"/>
+        </inertial>
     </link>
     <joint name="right_wheel_joint" type="continuous">
@@ -52,4 +92,17 @@
             <origin xyz="0 0 0" rpy="0 0 0"/>
         </visual>
+        <collision>
+            <origin xyz="0 0 0" rpy="0 0 0"/>
+            <geometry>
+                    <sphere radius="0.005"/>
+            </geometry>
+        </collision>
+        <inertial>
+            <origin xyz="3.89968128948481E-07 2.40073004698083E-07 0.00219173397061506" rpy="0 0 0"/>
+            <mass value="1.44379265037903E-06"/>
+            <inertia ixx="7.23075276010246E-11" ixy="-6.10956883467859E-16"
+                    ixz="2.22849693525031E-15" iyy="3.8713793085917E-11"
+                    iyz="2.93909858781952E-15" izz="1.00967486676306E-10"/>
+        </inertial>
     </link>
     <joint name="castor_front_joint" type="fixed">
@@ -65,4 +118,17 @@
             <origin xyz="0 0 0" rpy="0 0 0"/>
         </visual>
+        <collision>
+            <origin xyz="0 0 0" rpy="0 0 0"/>
+            <geometry>
+                    <sphere radius="0.005"/>
+            </geometry>
+        </collision>
+        <inertial>
+            <origin xyz="3.8996812895542E-07 2.40073004698083E-07 0.00219173397061509" rpy="0 0 0"/>
+            <mass value="1.44379265037902E-06"/>
+            <inertia ixx="7.23075276010246E-11" ixy="-6.10956872363424E-16"
+                    ixz="2.22849693527207E-15" iyy="3.87137930859167E-11"
+                    iyz="2.939098587861E-15" izz="1.00967486676306E-10"/>
+        </inertial>
     </link>
     <joint name="castor_back_joint" type="fixed">
